File: fcb-kicad/i2c.kicad_sch (KiCad schematic)
At the start: 10 parts, among them J3 I2C, U4 QMC5883L, U8 BMP388

Commit message: PCB rev0: "Babby's first Leiska"
Parts:
- renumbered C21 to C17, C22 to C18, C23 to C21, J3 to J4, R9 to R21, R10 to R22, U8 to U7, U4 to U8
Changed lines of the file:
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@@
   (symbol (lib_id "power:GND") (at 102.87 113.03 0) (unit 1)
     (in_bom yes) (on_board yes) (fields_autoplaced)
-    (property "Reference" "#PWR0128" (id 0) (at 102.87 119.38 0)
+    (property "Reference" "#PWR063" (id 0) (at 102.87 119.38 0)
       (effects (font (size 1.27 1.27)) hide)
     )
@@
   (symbol (lib_id "Device:R_Small") (at 35.56 34.29 0) (unit 1)
     (in_bom yes) (on_board yes) (fields_autoplaced)
-    (property "Reference" "R9" (id 0) (at 37.0586 33.3815 0)
+    (property "Reference" "R21" (id 0) (at 37.0586 33.3815 0)
       (effects (font (size 1.27 1.27)) (justify left))
     )
@@
   (symbol (lib_id "power:+3.3V") (at 35.56 31.75 0) (unit 1)
     (in_bom yes) (on_board yes) (fields_autoplaced)
-    (property "Reference" "#PWR021" (id 0) (at 35.56 35.56 0)
+    (property "Reference" "#PWR054" (id 0) (at 35.56 35.56 0)
       (effects (font (size 1.27 1.27)) hide)
     )
@@
   (symbol (lib_id "000_sjt:BMP388") (at 74.93 105.41 0) (unit 1)
     (in_bom yes) (on_board yes)
-    (property "Reference" "U8" (id 0) (at 74.93 85.09 0))
+    (property "Reference" "U7" (id 0) (at 74.93 85.09 0))
     (property "Value" "BMP388" (id 1) (at 74.93 87.63 0))
     (property "Footprint" "000_sjt:PQFN50P200X200X80-10N" (id 2) (at 74.93 146.05 0)
@@
   (symbol (lib_id "power:GND") (at 66.04 43.18 0) (unit 1)
     (in_bom yes) (on_board yes) (fields_autoplaced)
-    (property "Reference" "#PWR031" (id 0) (at 66.04 49.53 0)
+    (property "Reference" "#PWR059" (id 0) (at 66.04 49.53 0)
       (effects (font (size 1.27 1.27)) hide)
     )
@@
   (symbol (lib_id "Device:C_Small") (at 102.87 105.41 0) (unit 1)
     (in_bom yes) (on_board yes) (fields_autoplaced)
-    (property "Reference" "C21" (id 0) (at 105.1941 104.5078 0)
+    (property "Reference" "C17" (id 0) (at 105.1941 104.5078 0)
       (effects (font (size 1.27 1.27)) (justify left))
     )
@@
   (symbol (lib_id "power:+3V3") (at 116.84 97.79 0) (unit 1)
     (in_bom yes) (on_board yes) (fields_autoplaced)
-    (property "Reference" "#PWR0130" (id 0) (at 116.84 101.6 0)
+    (property "Reference" "#PWR064" (id 0) (at 116.84 101.6 0)
       (effects (font (size 1.27 1.27)) hide)
     )
@@
   (symbol (lib_id "power:+3.3V") (at 43.18 31.75 0) (unit 1)
     (in_bom yes) (on_board yes) (fields_autoplaced)
-    (property "Reference" "#PWR024" (id 0) (at 43.18 35.56 0)
+    (property "Reference" "#PWR055" (id 0) (at 43.18 35.56 0)
       (effects (font (size 1.27 1.27)) hide)
     )
@@
   (symbol (lib_id "power:GND") (at 189.23 123.19 0) (unit 1)
     (in_bom yes) (on_board yes) (fields_autoplaced)
-    (property "Reference" "#PWR0131" (id 0) (at 189.23 129.54 0)
+    (property "Reference" "#PWR067" (id 0) (at 189.23 129.54 0)
       (effects (font (size 1.27 1.27)) hide)
     )
@@
   (symbol (lib_id "Connector_Generic:Conn_01x04") (at 73.66 39.37 0) (mirror x) (unit 1)
     (in_bom yes) (on_board yes)
-    (property "Reference" "J3" (id 0) (at 73.66 29.0535 0))
+    (property "Reference" "J4" (id 0) (at 73.66 29.0535 0))
     (property "Value" "I2C" (id 1) (at 73.66 31.75 0))
     (property "Footprint" "Connector_PinHeader_2.00mm:PinHeader_1x04_P2.00mm_Vertical" (id 2) (at 73.66 39.37 0)
@@
   (symbol (lib_id "power:GND") (at 116.84 113.03 0) (unit 1)
     (in_bom yes) (on_board yes) (fields_autoplaced)
-    (property "Reference" "#PWR0126" (id 0) (at 116.84 119.38 0)
+    (property "Reference" "#PWR065" (id 0) (at 116.84 119.38 0)
       (effects (font (size 1.27 1.27)) hide)
     )
@@
   (symbol (lib_id "power:+3V3") (at 187.96 86.36 0) (unit 1)
     (in_bom yes) (on_board yes) (fields_autoplaced)
-    (property "Reference" "#PWR051" (id 0) (at 187.96 90.17 0)
+    (property "Reference" "#PWR066" (id 0) (at 187.96 90.17 0)
       (effects (font (size 1.27 1.27)) hide)
     )
@@
   (symbol (lib_id "power:+3V3") (at 102.87 97.79 0) (unit 1)
     (in_bom yes) (on_board yes) (fields_autoplaced)
-    (property "Reference" "#PWR0129" (id 0) (at 102.87 101.6 0)
+    (property "Reference" "#PWR062" (id 0) (at 102.87 101.6 0)
       (effects (font (size 1.27 1.27)) hide)
     )
@@
   (symbol (lib_id "000_sjt:QMC5883L") (at 186.69 105.41 0) (unit 1)
     (in_bom yes) (on_board yes)
-    (property "Reference" "U4" (id 0) (at 194.945 89.2999 0)
+    (property "Reference" "U8" (id 0) (at 194.945 89.2999 0)
       (effects (font (size 1.27 1.27)) (justify left))
     )
@@
   (symbol (lib_id "Device:C_Small") (at 116.84 105.41 0) (unit 1)
     (in_bom yes) (on_board yes) (fields_autoplaced)
-    (property "Reference" "C22" (id 0) (at 119.1641 104.5078 0)
+    (property "Reference" "C18" (id 0) (at 119.1641 104.5078 0)
       (effects (font (size 1.27 1.27)) (justify left))
     )
@@
   (symbol (lib_id "power:GND") (at 91.44 120.65 0) (unit 1)
     (in_bom yes) (on_board yes) (fields_autoplaced)
-    (property "Reference" "#PWR0125" (id 0) (at 91.44 127 0)
+    (property "Reference" "#PWR060" (id 0) (at 91.44 127 0)
       (effects (font (size 1.27 1.27)) hide)
     )
@@
   (symbol (lib_id "power:GND") (at 60.96 113.03 0) (unit 1)
     (in_bom yes) (on_board yes) (fields_autoplaced)
-    (property "Reference" "#PWR0123" (id 0) (at 60.96 119.38 0)
+    (property "Reference" "#PWR057" (id 0) (at 60.96 119.38 0)
       (effects (font (size 1.27 1.27)) hide)
     )
@@
   (symbol (lib_id "Device:R_Small") (at 43.18 34.29 0) (unit 1)
     (in_bom yes) (on_board yes) (fields_autoplaced)
-    (property "Reference" "R10" (id 0) (at 44.6786 33.3815 0)
+    (property "Reference" "R22" (id 0) (at 44.6786 33.3815 0)
       (effects (font (size 1.27 1.27)) (justify left))
     )
@@
   (symbol (lib_id "power:GND") (at 204.47 123.19 0) (unit 1)
     (in_bom yes) (on_board yes) (fields_autoplaced)
-    (property "Reference" "#PWR053" (id 0) (at 204.47 129.54 0)
+    (property "Reference" "#PWR068" (id 0) (at 204.47 129.54 0)
       (effects (font (size 1.27 1.27)) hide)
     )
@@
   (symbol (lib_id "power:+3V3") (at 59.69 97.79 0) (unit 1)
     (in_bom yes) (on_board yes) (fields_autoplaced)
-    (property "Reference" "#PWR0124" (id 0) (at 59.69 101.6 0)
+    (property "Reference" "#PWR056" (id 0) (at 59.69 101.6 0)
       (effects (font (size 1.27 1.27)) hide)
     )
@@
     (pin "1")
   )
-  (symbol (lib_id "Device:C_Small") (at 226.06 105.41 0) (unit 1)
-    (in_bom yes) (on_board yes) (fields_autoplaced)
-    (property "Reference" "C23" (id 0) (at 228.3841 104.5078 0)
-      (effects (font (size 1.27 1.27)) (justify left))
+  (symbol (lib_id "Device:C_Small") (at 226.06 105.41 0) (mirror y) (unit 1)
+    (in_bom yes) (on_board yes) (fields_autoplaced)
+    (property "Reference" "C21" (id 0) (at 228.3841 104.5078 0)
+      (effects (font (size 1.27 1.27)) (justify right))
     )
     (property "Value" "100n" (id 1) (at 228.3841 107.2829 0)
-      (effects (font (size 1.27 1.27)) (justify left))
+      (effects (font (size 1.27 1.27)) (justify right))
     )
     (property "Footprint" "Capacitor_SMD:C_0603_1608Metric" (id 2) (at 226.06 105.41 0)
@@
   (symbol (lib_id "power:+3V3") (at 226.06 97.79 0) (unit 1)
     (in_bom yes) (on_board yes) (fields_autoplaced)
-    (property "Reference" "#PWR0132" (id 0) (at 226.06 101.6 0)
+    (property "Reference" "#PWR069" (id 0) (at 226.06 101.6 0)
       (effects (font (size 1.27 1.27)) hide)
     )
@@
   (symbol (lib_id "power:+3.3V") (at 66.04 33.02 0) (unit 1)
     (in_bom yes) (on_board yes) (fields_autoplaced)
-    (property "Reference" "#PWR025" (id 0) (at 66.04 36.83 0)
+    (property "Reference" "#PWR058" (id 0) (at 66.04 36.83 0)
       (effects (font (size 1.27 1.27)) hide)
     )
@@
   (symbol (lib_id "power:+3V3") (at 93.98 91.44 0) (unit 1)
     (in_bom yes) (on_board yes) (fields_autoplaced)
-    (property "Reference" "#PWR0127" (id 0) (at 93.98 95.25 0)
+    (property "Reference" "#PWR061" (id 0) (at 93.98 95.25 0)
       (effects (font (size 1.27 1.27)) hide)
     )
@@
   (symbol (lib_id "power:GND") (at 226.06 113.03 0) (unit 1)
     (in_bom yes) (on_board yes) (fields_autoplaced)
-    (property "Reference" "#PWR0133" (id 0) (at 226.06 119.38 0)
-      (effects (font (size 1.27 1.27)) hide)
-    )
+    (property "Reference" "#PWR070" (id 0) (at 226.06 119.38 0)
+      (effects (font (size 1.27 1.27)) hide)
+    )

Commit message: Less routing on inner layers, fabrication, BOM should be OK
Parts:
- removed C17: 100n, Capacitor_SMD:C_0603_1608Metric, symbol Device:C_Small
- removed U7: BMP388, 000_sjt:PQFN50P200X200X80-10N, symbol 000_sjt:BMP388
- added U7: DPS310, 000_sjt:PG-VLGA-8-1, symbol 000_sjt:DPS310
- C18, C21: LCSC (none) -> C14663
- C19: LCSC (none) -> C19666
- C20: LCSC (none) -> C21120
- J4: value I2C -> PH1X4; LCSC (none) -> C388723
- U8: LCSC (none) -> C976032
- renumbered R21 to R20, R22 to R21
Connections:
- net +3V3: now also U7.6 (VDDIO), U7.8 (VDD)
- net GND: now also U7.1 (GND), U7.7 (GND)
- net I2C1_SCL: now also U7.4 (SCK)
- net I2C1_SDA: now also U7.3 (SDI)
- no-connect marks 2 -> 3
Other:
- note added: "CLK up to 3.4 MHz"
- note added: "SDO in I2c mode = address select floating -> 0x76"
- note added: "Same supply for VDD, VDDIO and pins are very close -> 1 cap should be enough"
- note removed: "SDO: I2c Address set VSS -> 1110110 = 0x76"
- note removed: "VDD"
- note removed: "VDDIO"
- note removed: "up to 3.4 MHz"
- moved on the sheet: C18
