File: fcb-kicad/fcb.kicad_pcb (KiCad board)
At the start: 4 copper layers, 45 x 45 mm, 26 parts, among them Q1 S8050 J3Y, U1 TPS5430DDA, U2 AMS1117-3.3, U3 DL-RTS4432, U4 LSM6DS3, U5 STM32F411CEUx, U6 W25Q128JVS

Commit message: hierarchic schemas, paljon muuta kivaa
Parts:
- removed D2: 1N4148W, Diode_SMD:D_SOD-123
- added C10: 100n, Capacitor_SMD:C_0603_1608Metric, F.Cu at (79.7, 55.4)
- added C11: 4u7, Capacitor_SMD:C_0603_1608Metric, F.Cu at (56.5, 54.1)
- added C12: 100n, Capacitor_SMD:C_0603_1608Metric, F.Cu at (63.8, 45.6)
- added C13: 100n, Capacitor_SMD:C_0603_1608Metric, F.Cu at (47.7, 56.0)
- added C14: 100n, Capacitor_SMD:C_0603_1608Metric, F.Cu at (55.4, 49.1)
- added C15: 100n, Capacitor_SMD:C_0603_1608Metric, F.Cu at (43.7, 56.0)
- added C8: 4u7, Capacitor_SMD:C_0603_1608Metric, F.Cu at (52.5, 55.1)
- added C9: 100n, Capacitor_SMD:C_0603_1608Metric, F.Cu at (98.7, 47.6)
- added D6: 1N4148W, Diode_SMD:D_SOD-123, F.Cu at (52.2, 62.3)
- added FB1: 500mA 600Ω@100M, Capacitor_SMD:C_0805_2012Metric, F.Cu at (56.7, 40.4)
- added FB2: 500mA 600Ω@100M, Capacitor_SMD:C_0805_2012Metric, F.Cu at (55.6, 46.3)
- added FB3: 500mA 600Ω@100M, Capacitor_SMD:C_0805_2012Metric, F.Cu at (62.5, 37.0)
- added R10: 3k, Resistor_SMD:R_0603_1608Metric, F.Cu at (51.4, 69.7)
- added R11: 470, Resistor_SMD:R_0603_1608Metric, F.Cu at (51.4, 72.2)
- added R12: 3k, Resistor_SMD:R_0603_1608Metric, F.Cu at (57.1, 61.9)
- added R5: 10k, Resistor_SMD:R_0603_1608Metric, F.Cu at (61.0, 40.1)
- added R6: 10k, Resistor_SMD:R_0603_1608Metric, F.Cu at (69.0, 39.3)
- added R7: 10k, Resistor_SMD:R_0603_1608Metric, F.Cu at (65.0, 42.3)
- added R8: 3k, Resistor_SMD:R_0603_1608Metric, F.Cu at (66.7, 36.8)
- added R9: 3k, Resistor_SMD:R_0603_1608Metric, F.Cu at (56.3, 65.2)
- added U3: DL-RTS4432, 000_sjt:DL-RTS4432_board, F.Cu at (87.2, 45.6)
- added U7: LSM6DS3, Package_LGA:LGA-14_3x2.5mm_P0.5mm_LayoutBorder3x4y, F.Cu at (109.3, 37.5)
- added U8: BMP388, 000_sjt:PQFN50P200X200X80-10N, F.Cu at (79.9, 61.4)
- C1: value 10u -> 10u 50V; footprint Capacitor_SMD:C_1206_3216Metric_Pad1.33x1.80mm_HandSolder -> Capacitor_SMD:C_1206_3216Metric
- C2: value 100n -> 100n 50V; footprint Capacitor_SMD:C_0603_1608Metric_Pad1.08x0.95mm_HandSolder -> Capacitor_SMD:C_0603_1608Metric
- C5: footprint Capacitor_SMD:C_0603_1608Metric_Pad1.08x0.95mm_HandSolder -> Capacitor_SMD:C_0603_1608Metric
- C6, C7: footprint Capacitor_SMD:C_1206_3216Metric_Pad1.33x1.80mm_HandSolder -> Capacitor_SMD:C_0603_1608Metric
- R4: value 470 -> 3k
- moved U5 153.8 mm to (49.9, 40.2)
- moved R4 145.5 mm to (59.8, 45.6)
- moved Q1 144.8 mm to (51.8, 66.2)
- moved BZ1 144.0 mm to (40.0, 67.5)
- moved D1 123.6 mm to (57.4, 37.2)
- moved C1 120.8 mm to (47.6, 53.0)
- moved R2 120.5 mm to (56.5, 43.1)
- moved C2 118.8 mm to (60.5, 43.1)
- moved C3 116.0 mm to (65.0, 39.8)
- moved L1 116.0 mm to (40.1, 48.2)
- moved C4 115.4 mm to (38.6, 54.8)
- moved R1 115.1 mm to (70.7, 36.8)
- moved C5 113.5 mm to (56.5, 51.6)
- moved R3 112.9 mm to (69.0, 41.8)
- moved C7 111.7 mm to (59.8, 48.1)
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Connections:
- net +BATT renamed Net-(C1-Pad2)
- C1 pad 1: -BATT -> GND
- C2 pad 1: -BATT -> GND
- C4 pad 2: -BATT -> GND
- C5 pad 1: -BATT -> GND
- C6 pad 1: -BATT -> GND
- C7 pad 1: -BATT -> GND
- D1 pad 2: -BATT -> GND
- Q1 pad 2: unconnected-(Q1-Pad2) -> GND
- R3 pad 2: -BATT -> GND
- R4 pad 1: BUZZER -> Net-(D2-Pad1)
- R4 pad 2: Net-(Q1-Pad1) -> GND
- U1 pad 6: -BATT -> GND
- U1 pad 9: -BATT -> GND
- U2 pad 1: -BATT -> GND
- U3 pad 13: unconnected-(U3-Pad13) -> RAD_CS_N
- U3 pad 14: unconnected-(U3-Pad14) -> RAD_IRQ_N
- U3 pad 6: unconnected-(U3-Pad6) -> RAD_GPIO_0
- U5 pad 1: unconnected-(U5-Pad1) -> +3V3
- U5 pad 10: unconnected-(U5-Pad10) -> AI_VBAT
- U5 pad 11: unconnected-(U5-Pad11) -> AI_CRNT
- U5 pad 12: unconnected-(U5-Pad12) -> AI_5V_1
- U5 pad 13: unconnected-(U5-Pad13) -> AI_5V_2
- U5 pad 14: unconnected-(U5-Pad14) -> AI_3V
- U5 pad 15: unconnected-(U5-Pad15) -> SPI1_SCK
- U5 pad 16: unconnected-(U5-Pad16) -> SPI1_MISO
- U5 pad 17: unconnected-(U5-Pad17) -> SPI1_MOSI
- U5 pad 18: unconnected-(U5-Pad18) -> TIM3_CH3
- U5 pad 19: unconnected-(U5-Pad19) -> TIM3_CH4
- U5 pad 2: unconnected-(U5-Pad2) -> RAD_IRQ_N
- U5 pad 20: unconnected-(U5-Pad20) -> IMU_CS
- U5 pad 21: unconnected-(U5-Pad21) -> SPI2_SCK
- U5 pad 22: unconnected-(U5-Pad22) -> Net-(U5-Pad22)
- U5 pad 23: unconnected-(U5-Pad23) -> GND
- U5 pad 24: unconnected-(U5-Pad24) -> +3V3
- U5 pad 25: unconnected-(U5-Pad25) -> IMU_INT1
- U5 pad 26: unconnected-(U5-Pad26) -> GPIO_PB13
- U5 pad 27: unconnected-(U5-Pad27) -> SPI2_MISO
- U5 pad 28: unconnected-(U5-Pad28) -> SPI2_MOSI
- U5 pad 29: unconnected-(U5-Pad29) -> FLASH_CS_N
- U5 pad 3: unconnected-(U5-Pad3) -> RAD_CS_N
- U5 pad 30: unconnected-(U5-Pad30) -> USART1_TX
- U5 pad 31: unconnected-(U5-Pad31) -> USART1_RX
- U5 pad 32: unconnected-(U5-Pad32) -> USB_DM
- U5 pad 33: unconnected-(U5-Pad33) -> USB_DP
- U5 pad 34: unconnected-(U5-Pad34) -> SWDIO
- U5 pad 35: unconnected-(U5-Pad35) -> GND
- U5 pad 36: unconnected-(U5-Pad36) -> +3V3
- U5 pad 37: unconnected-(U5-Pad37) -> SWCLK
- U5 pad 38: unconnected-(U5-Pad38) -> BUZZER
- U5 pad 39: unconnected-(U5-Pad39) -> SWO
- U5 pad 4: unconnected-(U5-Pad4) -> RAD_GPIO_0
- U5 pad 40: unconnected-(U5-Pad40) -> TIM3_CH1
- U5 pad 41: unconnected-(U5-Pad41) -> TIM3_CH2
- U5 pad 42: unconnected-(U5-Pad42) -> I2C1_SCL
- U5 pad 43: unconnected-(U5-Pad43) -> I2C1_SDA
- U5 pad 44: unconnected-(U5-Pad44) -> CPU_BOOT0
- U5 pad 45: unconnected-(U5-Pad45) -> GPIO_PB8
- U5 pad 46: unconnected-(U5-Pad46) -> GPIO_PB9
- U5 pad 47: unconnected-(U5-Pad47) -> GND
- U5 pad 48: unconnected-(U5-Pad48) -> +3V3
- U5 pad 49: unconnected-(U5-Pad49) -> GND
- U5 pad 5: unconnected-(U5-Pad5) -> OSC_IN
- U5 pad 6: unconnected-(U5-Pad6) -> OSC_OUT
- U5 pad 7: unconnected-(U5-Pad7) -> CPU_NRST
- U5 pad 8: unconnected-(U5-Pad8) -> GNDA
- U5 pad 9: unconnected-(U5-Pad9) -> +3.3VA
Routing:
- added copper zone on B.Cu, net GND
- added copper zone on F.Cu, net GND
- removed copper zone on B.Cu, net -BATT
- removed copper zone on F.Cu, net -BATT

Commit message: buzzer footprint
Parts:
- removed the U3 at (87.2, 45.6)
- removed the U3 at (147.2, 100.8)
- added C18: 100n, Capacitor_SMD:C_0603_1608Metric, F.Cu at (94.0, 68.2)
- added D2: LED_red, LED_SMD:LED_0603_1608Metric, F.Cu at (72.4, 85.0)
- added D3: LED_red, LED_SMD:LED_0603_1608Metric, F.Cu at (72.4, 87.6)
- added D4: B5819W SL, Diode_SMD:D_SOD-123, F.Cu at (67.5, 85.4)
- added D5: Blue, 3V, LED_SMD:LED_0603_1608Metric, F.Cu at (77.1, 76.0)
- added D6: Blue, 3V, LED_SMD:LED_0603_1608Metric, F.Cu at (66.7, 78.6)
- added D7: 1N4148W, Diode_SMD:D_SOD-123, F.Cu at (77.9, 68.6)
- added Q1: S8050 J3Y, Package_TO_SOT_SMD:SOT-23, F.Cu at (83.2, 69.2)
- added R10: 10k, Resistor_SMD:R_0603_1608Metric, F.Cu at (83.8, 84.9)
- added R11: 10k, Resistor_SMD:R_0603_1608Metric, F.Cu at (82.2, 72.6)
- added R12: 240, Resistor_SMD:R_0603_1608Metric, F.Cu at (70.7, 78.6)
- added R17: 240, Resistor_SMD:R_0603_1608Metric, F.Cu at (74.7, 78.6)
- added R18: 470, Resistor_SMD:R_0603_1608Metric, F.Cu at (81.1, 76.0)
- added R9: 10k, Resistor_SMD:R_0603_1608Metric, F.Cu at (79.8, 84.9)
- added U3: DL-RTS4432, 000_sjt:DL-RTS4432_board, B.Cu at (69.5, 109.5)
- added U9: USBLC6-2SC6, Package_TO_SOT_SMD:SOT-23-6, F.Cu at (77.6, 72.5)
- BZ1: footprint Buzzer_Beeper:Buzzer_TDK_PS1240P02BT_D12.2mm_H6.5mm -> 000_sjt:MLT-8350
- H1, H2, H3, H4: footprint MountingHole:MountingHole_3.2mm_M3 -> MountingHole:MountingHole_3.2mm_M3_DIN965_Pad
- moved BZ1 63.0 mm to (94.0, 100.0)
- moved H1 30.0 mm to (161.5, 116.5)
- moved H2 30.0 mm to (131.5, 116.5)
- moved H3 30.0 mm to (131.5, 86.5)
- moved H4 30.0 mm to (161.5, 86.5)
Connections:
- net IMU_CS renamed IMU_CS_N
- BZ1 pad 2: Net-(BZ1-Pad2) -> /IO/Buzzer_-
- C10 pad 1: Net-(C10-Pad1) -> CPU_VDD
- C10 pad 2: +3V3 -> GND
- C11 pad 2: +3V3 -> CPU_VDD
- C12 pad 2: +3V3 -> CPU_VDD
- C13 pad 2: +3V3 -> CPU_VDD
- C14 pad 2: +3V3 -> CPU_VDD
- C15 pad 2: +3V3 -> CPU_VDD
- C7 pad 2: +3V3 -> CPU_VDD
- C9 pad 1: Net-(C9-Pad1) -> CPU_VDD
- C9 pad 2: +3V3 -> GND
- FB3 pad 1: +3V3 -> CPU_VDD
- R5 pad 1: +3V3 -> CPU_VDD
- R6 pad 1: +3V3 -> CPU_VDD
- U2 pad 2: +3V3 -> CPU_VDD
- U5 pad 1: +3V3 -> CPU_VDD
- U5 pad 24: +3V3 -> CPU_VDD
- U5 pad 36: +3V3 -> CPU_VDD
- U5 pad 48: +3V3 -> CPU_VDD
- U6 pad 1: unconnected-(U6-Pad1) -> FLASH_CS_N
- U6 pad 2: unconnected-(U6-Pad2) -> SPI2_MISO
- U6 pad 3: unconnected-(U6-Pad3) -> Net-(R24-Pad2)
- U6 pad 4: unconnected-(U6-Pad4) -> GND
- U6 pad 5: unconnected-(U6-Pad5) -> SPI2_MOSI
- U6 pad 6: unconnected-(U6-Pad6) -> SPI2_SCK
- U6 pad 7: unconnected-(U6-Pad7) -> Net-(R25-Pad2)
- U6 pad 8: unconnected-(U6-Pad8) -> CPU_VDD
- U7 pad 1: IMU_SDO -> SPI1_MISO
- U7 pad 13: IMU_SPC -> SPI1_SCK
- U7 pad 14: IMU_SDI -> SPI1_MOSI
- U7 pad 5: Net-(C9-Pad1) -> CPU_VDD
- U7 pad 8: Net-(C10-Pad1) -> CPU_VDD
- U7 pad 9: IMU_INT2 -> unconnected-(U7-Pad9)

Commit message: Schema rev0 done, Layout components grouped
Parts:
- removed the D6 at (66.7, 78.6)
- removed the D6 at (52.2, 62.3)
- removed FB2, FB3: 500mA 600Ω@100M, Capacitor_SMD:C_0805_2012Metric
- removed the Q1 at (51.8, 66.2)
- removed the Q1 at (83.2, 69.2)
- removed the R10 at (51.4, 69.7)
- removed the R10 at (83.8, 84.9)
- removed the R11 at (82.2, 72.6)
- removed the R11 at (51.4, 72.2)
- removed the R12 at (57.1, 61.9)
- removed the R12 at (70.7, 78.6)
- removed the R9 at (56.3, 65.2)
- removed the R9 at (79.8, 84.9)
- added C19: 4.7u, Capacitor_SMD:C_0603_1608Metric, F.Cu at (96.0, 154.0)
- added C20: 220n, Capacitor_SMD:C_0603_1608Metric, F.Cu at (94.5, 153.5)
- added C21: 100n, Capacitor_SMD:C_0603_1608Metric, F.Cu at (242.0, 116.5)
- added C22: 100n, Capacitor_SMD:C_0603_1608Metric, F.Cu at (241.5, 111.0)
- added C23: 100n, Capacitor_SMD:C_0603_1608Metric, F.Cu at (92.5, 150.0)
- added CL1: 8p, Capacitor_SMD:C_0603_1608Metric, F.Cu at (103.0, 65.0)
- added CL2: 8p, Capacitor_SMD:C_0603_1608Metric, F.Cu at (103.0, 73.0)
- added D6: Blue, 3V, LED_SMD:LED_0603_1608Metric, F.Cu at (266.5, 79.5)
- added J1: Conn_ESC_4in1, Connector_JST:JST_SH_SM08B-SRSS-TB_1x08-1MP_P1.00mm_Horizontal, F.Cu at (147.8, 73.0)
- added J10: Conn_Coaxial, 000_sjt:KH-IPEX-K501-29, B.Cu at (138.5, 149.0)
- added J11: UART, Connector_PinHeader_2.00mm:PinHeader_1x04_P2.00mm_Vertical, F.Cu at (275.5, 126.0)
- added J2: SWD, Connector_PinHeader_1.27mm:PinHeader_2x05_P1.27mm_Vertical, F.Cu at (270.4, 93.5)
- added J3: I2C, Connector_PinHeader_2.00mm:PinHeader_1x04_P2.00mm_Vertical, F.Cu at (264.5, 134.0)
- added J4: USB_B_Micro, 000_omat:MICRO-USB-SMD_U254-051T-4BH83-F1S, F.Cu at (134.0, 58.0)
- added J5: PB9, Connector_PinHeader_2.00mm:PinHeader_1x03_P2.00mm_Vertical, F.Cu at (214.0, 129.0)
- added J6: PB13, Connector_PinHeader_2.00mm:PinHeader_1x03_P2.00mm_Vertical, F.Cu at (269.5, 77.5)
- added J7: AI_5V_1, Connector_PinHeader_2.00mm:PinHeader_1x03_P2.00mm_Vertical, F.Cu at (269.5, 117.0)
- added J8: AI_5V_2, Connector_PinHeader_2.00mm:PinHeader_1x03_P2.00mm_Vertical, F.Cu at (264.8, 104.5)
- added J9: AI_3V, Connector_PinHeader_2.00mm:PinHeader_1x03_P2.00mm_Vertical, F.Cu at (271.5, 127.5)
- added Q1: S8050 J3Y, Package_TO_SOT_SMD:SOT-23, F.Cu at (274.5, 153.0)
- added R10: 10k, Resistor_SMD:R_0603_1608Metric, F.Cu at (83.5, 74.0)
- added R11: 10k, Resistor_SMD:R_0603_1608Metric, F.Cu at (226.5, 150.5)
- added R12: 240, Resistor_SMD:R_0603_1608Metric, F.Cu at (208.0, 131.0)
- added R13: 22R, Resistor_SMD:R_0603_1608Metric, F.Cu at (265.6, 94.3)
- added R14: 22R, Resistor_SMD:R_0603_1608Metric, F.Cu at (265.6, 97.3)
- added R15: 22R, Resistor_SMD:R_0603_1608Metric, F.Cu at (265.6, 95.8)
- added R16: 22R, Resistor_SMD:R_0603_1608Metric, F.Cu at (265.6, 98.8)
- added R19: 10k, Resistor_SMD:R_0603_1608Metric, F.Cu at (91.0, 100.0)
- added R20: 10k, Resistor_SMD:R_0603_1608Metric, F.Cu at (241.0, 78.6)
- added R21: 10k, Resistor_SMD:R_0603_1608Metric, F.Cu at (139.5, 142.0)
- added R22: 10k, Resistor_SMD:R_0603_1608Metric, F.Cu at (265.7, 119.5)
- added R24: 10k, Resistor_SMD:R_0603_1608Metric, F.Cu at (92.5, 107.5)
- added R25: 10k, Resistor_SMD:R_0603_1608Metric, F.Cu at (95.5, 107.5)
- added R26: 10k, Resistor_SMD:R_0603_1608Metric, F.Cu at (211.0, 59.0)
- added R27: 1k, Resistor_SMD:R_0603_1608Metric, F.Cu at (210.7, 61.5)
- added R28: 1k, Resistor_SMD:R_0603_1608Metric, F.Cu at (102.0, 71.0)
- added R29: 10k, Resistor_SMD:R_0603_1608Metric, F.Cu at (265.5, 121.5)
- added R30: 10k, Resistor_SMD:R_0603_1608Metric, F.Cu at (268.5, 111.5)
- added R31: 10k, Resistor_SMD:R_0603_1608Metric, F.Cu at (265.5, 117.5)
- added R32: 5k, Resistor_SMD:R_0603_1608Metric, F.Cu at (265.3, 111.5)
- added R9: 10k, Resistor_SMD:R_0603_1608Metric, F.Cu at (85.0, 76.5)
- added SW1: SW_Push, 000_sjt:Button-2.9x4.0mm-SMD, F.Cu at (224.5, 155.0)
- added SW2: SW_SPDT, 000_sjt:DIP_SPDT, F.Cu at (210.0, 152.9)
- added SW3: BTN_USER, 000_sjt:Button-2.9x4.0mm-SMD, F.Cu at (225.0, 148.0)
- added Y1: 16 MHz, Crystal:Crystal_SMD_3225-4Pin_3.2x2.5mm, F.Cu at (102.5, 68.5)
- C11, C8: value 4u7 -> 4.7u
- C15: value 100n -> 10u
- C6: value 10u -> 100n
- R4, R8: value 3k -> 1k
- U1: footprint Package_SO:TI_SO-PowerPAD-8_ThermalVias -> Package_SO:TI_SO-PowerPAD-8
- U4: value LSM6DS3 -> QMC5883L; footprint Package_LGA:LGA-14_3x2.5mm_P0.5mm_LayoutBorder3x4y -> 000_sjt:QMC5883L
- moved D7 208.5 mm to (266.5, 157.5)
- moved R5 202.1 mm to (225.5, 157.5)
- moved R18 198.7 mm to (262.5, 157.0)
- moved R17 188.3 mm to (263.0, 79.5)
- moved C15 186.8 mm to (230.5, 52.0)
- moved R6 186.1 mm to (213.5, 156.5), turned to 180 degrees
- moved U2 185.0 mm to (225.1, 47.9)
- moved L1 184.3 mm to (224.0, 36.4)
- moved C4 182.4 mm to (221.0, 55.5)
- moved R4 182.2 mm to (242.0, 47.0)
- moved R7 179.0 mm to (209.0, 148.5)
- moved BZ1 178.5 mm to (265.5, 149.5)
- moved D3 175.5 mm to (242.0, 42.5)
- moved R8 175.4 mm to (242.0, 44.0)
- moved D2 173.8 mm to (242.5, 49.5)
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Connections:
- net /IO/Buzzer_- renamed /IO/Q_buzzzer_C
- net Net-(C1-Pad2) renamed /VIN
- net Net-(C3-Pad1) renamed /BOOT
- net Net-(C3-Pad2) renamed /PH
- net Net-(C8-Pad2) renamed /VCAP
- net Net-(R1-Pad2) renamed /VSENSE
- BZ1 pad 1: +5V -> +3V3
- C10 pad 1: CPU_VDD -> +3V3
- C11 pad 2: CPU_VDD -> +3V3
- C12 pad 2: CPU_VDD -> +3V3
- C13 pad 2: CPU_VDD -> +3V3
- C14 pad 2: CPU_VDD -> +3V3
- C15 pad 2: CPU_VDD -> +5V
- C18 pad 1: CPU_VDD -> +3V3
- C6 pad 2: +5V -> +3V3
- C7 pad 2: CPU_VDD -> +3V3
- C9 pad 1: CPU_VDD -> +3V3
- D3 pad 2: CPU_VDD -> +3V3
- D7 pad 1: +5V -> +3V3
- R18 pad 2: Net-(Q1-Pad1) -> /IO/Q_buzzer_B
- R5 pad 1: CPU_VDD -> +3V3
- R6 pad 1: CPU_VDD -> +3V3
- U2 pad 2: CPU_VDD -> +3V3
- U3 pad 1: unconnected-(U3-Pad1) -> /SPI peripherials/ANT
- U3 pad 5: CPU_VDD -> +3V3
- U4 pad 1: unconnected-(U4-Pad1) -> I2C1_SCL
- U4 pad 10: unconnected-(U4-Pad10) -> Net-(C19-Pad1)
- U4 pad 11: unconnected-(U4-Pad11) -> GND
- U4 pad 12: unconnected-(U4-Pad12) -> Net-(C20-Pad1)
- U4 pad 13: unconnected-(U4-Pad13) -> +3V3
- U4 pad 2: unconnected-(U4-Pad2) -> +3V3
- U4 pad 4: unconnected-(U4-Pad4) -> +3V3
- U4 pad 8: unconnected-(U4-Pad8) -> Net-(C20-Pad2)
- U4 pad 9: unconnected-(U4-Pad9) -> GND
- U5 pad 1: CPU_VDD -> +3V3
- U5 pad 12: AI_5V_1 -> AI_5V_3V_1
- U5 pad 13: AI_5V_2 -> AI_5V_3V_2
- U5 pad 24: CPU_VDD -> +3V3
- U5 pad 36: CPU_VDD -> +3V3
- U5 pad 48: CPU_VDD -> +3V3
- U5 pad 8: GNDA -> GND
- U5 pad 9: +3.3VA -> +3V3
- U6 pad 8: CPU_VDD -> +3V3
- U7 pad 5: CPU_VDD -> +3V3
- U7 pad 8: CPU_VDD -> +3V3
- U8 pad 1: unconnected-(U8-Pad1) -> +3V3
- U8 pad 10: unconnected-(U8-Pad10) -> +3V3
- U8 pad 2: unconnected-(U8-Pad2) -> I2C1_SCL
- U8 pad 3: Net-(U8-Pad3) -> GND
- U8 pad 4: unconnected-(U8-Pad4) -> I2C1_SDA
- U8 pad 5: unconnected-(U8-Pad5) -> GND
- U8 pad 6: unconnected-(U8-Pad6) -> +3V3
- U8 pad 8: Net-(U8-Pad3) -> GND
- U8 pad 9: Net-(U8-Pad3) -> GND
- U9 pad 4: Net-(J4-Pad3) -> /IO/USB_CONN+
- U9 pad 6: Net-(J4-Pad2) -> /IO/USB_CONN-
Routing:
- net /SPI peripherials/ANT: track 0.00 -> 4.20 mm
- net Net-(C19-Pad1): track 0.00 -> 2.95 mm
- net /VSENSE: track 0.00 -> 2.46 mm
- net Net-(C20-Pad2): track 0.00 -> 1.76 mm
- net SPI2_MOSI: track 0.00 -> 1.62 mm
- net Net-(C20-Pad1): track 0.00 -> 1.43 mm
- added copper zone on In1.Cu, net +3V3
- added copper zone on In2.Cu, net +5V

Commit message: PCB rev0: "Babby's first Leiska"
Parts:
- removed C22, C23: 100n, Capacitor_SMD:C_0603_1608Metric
- removed R12: 240, Resistor_SMD:R_0603_1608Metric
- removed R31: 10k, Resistor_SMD:R_0603_1608Metric
- removed R32: 5k, Resistor_SMD:R_0603_1608Metric
- removed SW2: SW_SPDT, 000_sjt:DIP_SPDT
- added C16: 100n, Capacitor_SMD:C_0603_1608Metric, B.Cu at (147.5, 104.2)
- added C17: 100n, Capacitor_SMD:C_0603_1608Metric, B.Cu at (157.0, 116.0)
- added R23: 10k, Resistor_SMD:R_0603_1608Metric, F.Cu at (133.8, 122.0)
- C1: value 10u 50V -> 4.7u; footprint Capacitor_SMD:C_1206_3216Metric -> Capacitor_SMD:C_0603_1608Metric
- C11: value 4.7u -> 100u 6.3V; footprint Capacitor_SMD:C_0603_1608Metric -> Capacitor_Tantalum_SMD:CP_EIA-3528-15_AVX-H_Pad1.50x2.35mm_HandSolder
- C12, C13: value 100n -> 10u
- C14, C18, C21, C5, C6: moved to B.Cu
- C15, C7: value 10u -> 100n; moved to B.Cu
- C2: value 100n 50V -> 10u 50V; footprint Capacitor_SMD:C_0603_1608Metric -> Capacitor_SMD:C_1206_3216Metric
- C3: value 10n -> 100n 50V
- C4: value 100u 6.3V -> 4.7u; footprint Capacitor_Tantalum_SMD:CP_EIA-3528-15_AVX-H_Pad1.50x2.35mm_HandSolder -> Capacitor_SMD:C_0603_1608Metric
- C8: value 4.7u -> 100n; moved to B.Cu
- C9: value 100n -> 10n
- D2: value LED_red -> B5819W SL; footprint LED_SMD:LED_0603_1608Metric -> Diode_SMD:D_SOD-123
- D4: value B5819W SL -> LED_red; footprint Diode_SMD:D_SOD-123 -> LED_SMD:LED_0603_1608Metric
- J10: value Conn_Coaxial -> AI_5V_2; footprint 000_sjt:KH-IPEX-K501-29 -> Connector_PinHeader_2.00mm:PinHeader_1x03_P2.00mm_Vertical; moved to F.Cu
- J11: value UART -> AI_3V; footprint Connector_PinHeader_2.00mm:PinHeader_1x04_P2.00mm_Vertical -> Connector_PinHeader_2.00mm:PinHeader_1x03_P2.00mm_Vertical
- J3: value I2C -> Conn_Coaxial; footprint Connector_PinHeader_2.00mm:PinHeader_1x04_P2.00mm_Vertical -> 000_sjt:KH-IPEX-K501-29; moved to B.Cu
- J4: value USB_B_Micro -> I2C; footprint 000_omat:MICRO-USB-SMD_U254-051T-4BH83-F1S -> Connector_PinHeader_2.00mm:PinHeader_1x04_P2.00mm_Vertical
- J5: value PB9 -> USB_B_Micro; footprint Connector_PinHeader_2.00mm:PinHeader_1x03_P2.00mm_Vertical -> 000_sjt:MICRO-USB-SMD_U254-051T-4BH83-F1S
- J6: value PB13 -> PB9
- J7: value AI_5V_1 -> PB13
- J8: value AI_5V_2 -> UART; footprint Connector_PinHeader_2.00mm:PinHeader_1x03_P2.00mm_Vertical -> Connector_PinHeader_2.00mm:PinHeader_1x04_P2.00mm_Vertical
- J9: value AI_3V -> AI_5V_1
- R10, R7, R9: value 10k -> 22R
- R13, R16: value 22R -> 10k
- R14, R15: value 22R -> 1k
- R17, R3: value 240 -> 10k
- R18: value 470 -> 10k
- R2: value 3k -> 1k
- R24, R25, R5: value 10k -> 240
- R26: value 10k -> 470
- R27: value 1k -> 5k
- R28: value 1k -> 10k
- R29: value 10k -> 5k
- R4: value 1k -> 3k
- R6: value 10k -> 1k
- R8: value 1k -> 22R
- U1: value TPS5430DDA -> STM32F411CEUx; footprint Package_SO:TI_SO-PowerPAD-8 -> Package_DFN_QFN:QFN-48-1EP_7x7mm_P0.5mm_EP5.6x5.6mm
- U2: value AMS1117-3.3 -> TPS5430DDA; footprint Package_TO_SOT_SMD:SOT-223-3_TabPin2 -> Package_SO:TI_SO-PowerPAD-8_ThermalVias
- U3: value DL-RTS4432 -> AMS1117-3.3; footprint 000_sjt:DL-RTS4432_board -> Package_TO_SOT_SMD:SOT-223-3_TabPin2; moved to F.Cu
- U4: value QMC5883L -> W25Q128JVS; footprint 000_sjt:QMC5883L -> Package_SO:SOIC-8_5.23x5.23mm_P1.27mm
- U5: value STM32F411CEUx -> LSM6DS3; footprint Package_DFN_QFN:QFN-48-1EP_7x7mm_P0.5mm_EP5.6x5.6mm -> Package_LGA:LGA-14_3x2.5mm_P0.5mm_LayoutBorder3x4y
- U6: value W25Q128JVS -> DL-RTS4432; footprint Package_SO:SOIC-8_5.23x5.23mm_P1.27mm -> 000_sjt:DL-RTS4432_board; moved to B.Cu
- U7: value LSM6DS3 -> BMP388; footprint Package_LGA:LGA-14_3x2.5mm_P0.5mm_LayoutBorder3x4y -> 000_sjt:PQFN50P200X200X80-10N
- U8: value BMP388 -> QMC5883L; footprint 000_sjt:PQFN50P200X200X80-10N -> 000_sjt:QMC5883L
- moved J7 142.5 mm to (127.0, 113.8), turned to 180 degrees
- moved D6 140.3 mm to (129.5, 109.8), turned to 90 degrees
- moved R15 134.2 mm to (132.5, 112.2), turned to 180 degrees
- moved R14 133.7 mm to (132.4, 109.2), turned to 180 degrees
- moved R18 133.5 mm to (138.2, 108.2), turned to -90 degrees
- moved Q1 132.9 mm to (153.8, 97.5), turned to 90 degrees
- moved J8 129.9 mm to (136.2, 123.0), turned to 90 degrees
- moved D7 129.2 mm to (154.5, 93.0), turned to -90 degrees
- moved R17 128.8 mm to (139.4, 115.6)
- moved R16 127.1 mm to (139.4, 113.8), turned to 0 degrees
- moved D3 125.5 mm to (135.8, 109.2)
- moved J2 125.2 mm to (148.6, 122.8), turned to 180 degrees
- moved J3 120.7 mm to (154.0, 85.5), turned to 180 degrees
- moved BZ1 118.1 mm to (160.8, 95.0)
- moved R8 117.8 mm to (151.2, 119.2), turned to 90 degrees
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Connections:
- C1 pad 2: /VIN -> /VCAP
- C10 pad 1: +3V3 -> GND
- C10 pad 2: GND -> +5V
- C11 pad 1: GND -> +5V
- C11 pad 2: +3V3 -> GND
- C12 pad 2: +3V3 -> +5V
- C14 pad 1: GND -> +3V3
- C14 pad 2: +3V3 -> GND
- C15 pad 1: GND -> +3V3
- C15 pad 2: +5V -> GND
- C3 pad 1: /BOOT -> GND
- C3 pad 2: /PH -> /VIN
- C4 pad 1: +5V -> GND
- C4 pad 2: GND -> +3V3
- C5 pad 2: +5V -> +3V3
- C8 pad 2: /VCAP -> +3V3
- C9 pad 1: +3V3 -> /BOOT
- C9 pad 2: GND -> /PH
- CL2 pad 2: Net-(CL2-Pad2) -> /OSC_OUT_R
- D2 pad 1: Net-(D2-Pad1) -> +5V
- D2 pad 2: +5V -> 5V_USB
- D3 pad 2: +3V3 -> +5V
- D4 pad 1: +5V -> Net-(D4-Pad1)
- D4 pad 2: 5V_USB -> +3V3
- J10 pad 1: /SPI peripherials/ANT -> GND
- J10 pad 2: GND -> /IO/AI_5V_2
- J11 pad 2: USART1_TX -> AI_3V
- J11 pad 3: USART1_RX -> +3V3
- J3 pad 1: GND -> /SPI peripherials/ANT
- J3 pad 2: I2C1_SDA -> GND
- J4 pad 1: 5V_USB -> GND
- J4 pad 2: /IO/USB_CONN- -> I2C1_SDA
- J4 pad 3: /IO/USB_CONN+ -> I2C1_SCL
- J4 pad 4: unconnected-(J4-Pad4) -> +3V3
- J5 pad 1: GND -> 5V_USB
- J5 pad 2: GPIO_PB9 -> /IO/USB_CONN-
- J5 pad 3: +3V3 -> /IO/USB_CONN+
- J6 pad 2: GPIO_PB13 -> GPIO_PB9
- J7 pad 2: /IO/AI_5V_1 -> GPIO_PB13
- J7 pad 3: +5V -> +3V3
- J8 pad 2: /IO/AI_5V_2 -> USART1_TX
- J8 pad 3: +5V -> USART1_RX
- J9 pad 2: AI_3V -> /IO/AI_5V_1
- J9 pad 3: +3V3 -> +5V
- R1 pad 1: +5V -> +BATT
- R1 pad 2: /VSENSE -> AI_VBAT
- R10 pad 1: +3V3 -> Net-(J2-Pad10)
- R10 pad 2: I2C1_SDA -> CPU_NRST
- R11 pad 2: GPIO_PB8 -> CPU_NRST
- R13 pad 1: Net-(J2-Pad2) -> CPU_BOOT0
- R13 pad 2: SWDIO -> GND
- R14 pad 1: Net-(J2-Pad4) -> Net-(D3-Pad1)
- R14 pad 2: SWCLK -> GND
- R15 pad 1: Net-(J2-Pad6) -> Net-(D4-Pad1)
- R15 pad 2: SWO -> GND
- R16 pad 1: Net-(J2-Pad10) -> +3V3
- R16 pad 2: CPU_NRST -> FLASH_CS_N
- R17 pad 1: Net-(D6-Pad1) -> +3V3
- R17 pad 2: GND -> Net-(R17-Pad2)
- R18 pad 1: BUZZER -> +3V3
- R18 pad 2: /IO/Q_buzzer_B -> Net-(R18-Pad2)
- R19 pad 2: FLASH_CS_N -> IMU_CS_N
- R2 pad 1: /VSENSE -> AI_VBAT
- R2 pad 2: Net-(R2-Pad2) -> GND
- R20 pad 2: IMU_CS_N -> RAD_CS_N
- R21 pad 2: RAD_CS_N -> I2C1_SCL
- R22 pad 1: /IO/AI_5V_1 -> +3V3
- R22 pad 2: AI_5V_3V_1 -> I2C1_SDA
- R24 pad 1: +3V3 -> Net-(D5-Pad1)
- R24 pad 2: Net-(R24-Pad2) -> GND
- R25 pad 1: +3V3 -> Net-(D6-Pad1)
- R25 pad 2: Net-(R25-Pad2) -> GND
- R26 pad 1: +BATT -> BUZZER
- R26 pad 2: AI_VBAT -> /IO/Q_buzzer_B
- R27 pad 1: AI_VBAT -> /IO/AI_5V_1
- R27 pad 2: GND -> AI_5V_3V_1
- R28 pad 1: Net-(CL2-Pad2) -> AI_5V_3V_1
- R28 pad 2: OSC_OUT -> GND
- R29 pad 1: AI_5V_3V_1 -> /IO/AI_5V_2
- R29 pad 2: GND -> AI_5V_3V_2
- R3 pad 1: Net-(R2-Pad2) -> +5V
- R3 pad 2: GND -> /VSENSE
- R4 pad 1: Net-(D2-Pad1) -> /VSENSE
- R4 pad 2: GND -> Net-(R4-Pad2)
- R5 pad 1: +3V3 -> Net-(R4-Pad2)
- R5 pad 2: CPU_NRST -> GND
- R6 pad 1: +3V3 -> /OSC_OUT_R
- R6 pad 2: Net-(R6-Pad2) -> OSC_OUT
- R7 pad 1: Net-(R7-Pad1) -> Net-(J2-Pad2)
- R7 pad 2: GND -> SWDIO
- R8 pad 1: Net-(D3-Pad1) -> Net-(J2-Pad4)
- R8 pad 2: GND -> SWCLK
- R9 pad 1: +3V3 -> Net-(J2-Pad6)
- R9 pad 2: I2C1_SCL -> SWO
- U1 pad 1: /BOOT -> +3V3
- U1 pad 2: unconnected-(U1-Pad2) -> RAD_IRQ_N
- U1 pad 3: unconnected-(U1-Pad3) -> RAD_CS_N
- U1 pad 4: /VSENSE -> RAD_GPIO_0
- U1 pad 5: unconnected-(U1-Pad5) -> OSC_IN
- U1 pad 6: GND -> OSC_OUT
- U1 pad 7: /VIN -> CPU_NRST
- U1 pad 8: /PH -> GND
- U1 pad 9: GND -> +3V3
- U2 pad 1: GND -> /BOOT
- U2 pad 2: +3V3 -> unconnected-(U2-Pad2)
- U2 pad 3: +5V -> unconnected-(U2-Pad3)
- U3 pad 1: /SPI peripherials/ANT -> GND
- U3 pad 2: GND -> +3V3
- U3 pad 3: unconnected-(U3-Pad3) -> +5V
- U4 pad 1: I2C1_SCL -> FLASH_CS_N
- U4 pad 2: +3V3 -> SPI2_MISO
- U4 pad 3: unconnected-(U4-Pad3) -> Net-(R17-Pad2)
- U4 pad 4: +3V3 -> GND
- U4 pad 5: unconnected-(U4-Pad5) -> SPI2_MOSI
- U4 pad 6: unconnected-(U4-Pad6) -> SPI2_SCK
- U4 pad 7: unconnected-(U4-Pad7) -> Net-(R18-Pad2)
- U4 pad 8: Net-(C20-Pad2) -> +3V3
- U5 pad 1: +3V3 -> SPI1_MISO
- U5 pad 10: AI_VBAT -> unconnected-(U5-Pad10)
- U5 pad 11: AI_CRNT -> unconnected-(U5-Pad11)
- U5 pad 12: AI_5V_3V_1 -> IMU_CS_N
- U5 pad 13: AI_5V_3V_2 -> SPI1_SCK
- U5 pad 14: AI_3V -> SPI1_MOSI
- U5 pad 2: RAD_IRQ_N -> GND
- U5 pad 3: RAD_CS_N -> GND
- U5 pad 4: RAD_GPIO_0 -> IMU_INT1
- U5 pad 5: OSC_IN -> +3V3
- U5 pad 6: OSC_OUT -> GND
- U5 pad 7: CPU_NRST -> GND
- U5 pad 8: GND -> +3V3
- U5 pad 9: +3V3 -> unconnected-(U5-Pad9)
- U6 pad 1: FLASH_CS_N -> /SPI peripherials/ANT
- U6 pad 2: SPI2_MISO -> GND
- U6 pad 3: Net-(R24-Pad2) -> unconnected-(U6-Pad3)
- U6 pad 4: GND -> unconnected-(U6-Pad4)
- U6 pad 5: SPI2_MOSI -> +3V3
- U6 pad 6: SPI2_SCK -> RAD_GPIO_0
- U6 pad 7: Net-(R25-Pad2) -> unconnected-(U6-Pad7)
- U6 pad 8: +3V3 -> unconnected-(U6-Pad8)
- U7 pad 1: SPI1_MISO -> +3V3
- U7 pad 10: unconnected-(U7-Pad10) -> +3V3
- U7 pad 2: GND -> I2C1_SCL
- U7 pad 4: IMU_INT1 -> I2C1_SDA
- U7 pad 5: +3V3 -> GND
- U7 pad 6: GND -> +3V3
- U7 pad 7: GND -> unconnected-(U7-Pad7)
- U7 pad 8: +3V3 -> GND
- U7 pad 9: unconnected-(U7-Pad9) -> GND
- U8 pad 1: +3V3 -> I2C1_SCL
- U8 pad 10: +3V3 -> Net-(C19-Pad1)
- U8 pad 2: I2C1_SCL -> +3V3
- U8 pad 3: GND -> unconnected-(U8-Pad3)
- U8 pad 4: I2C1_SDA -> +3V3
- U8 pad 5: GND -> unconnected-(U8-Pad5)
- U8 pad 6: +3V3 -> unconnected-(U8-Pad6)
- U8 pad 8: GND -> Net-(C20-Pad2)
- U9 pad 1: USB_DM -> USB_D-
- U9 pad 3: USB_DP -> USB_D+
- Y1 pad 1: Net-(CL2-Pad2) -> /OSC_OUT_R
Routing:
- net GND: track 0.00 -> 136.4 mm, vias 0 -> 37
- net +5V: track 0.00 -> 87.7 mm, vias 0 -> 2
- net +3V3: track 0.00 -> 70.9 mm, vias 0 -> 23
- net CPU_NRST: track 0.00 -> 58.1 mm, vias 0 -> 2
- net BUZZER: track 0.00 -> 53.8 mm, vias 0 -> 2
- net TIM3_CH1: track 0.00 -> 44.1 mm, vias 0 -> 2
- net AI_VBAT: track 0.00 -> 42.6 mm, vias 0 -> 2
- net TIM3_CH2: track 0.00 -> 42.3 mm, vias 0 -> 2
- net USB_D+: track 0.00 -> 41.2 mm, vias 0 -> 2
- net USB_D-: track 0.00 -> 38.1 mm, vias 0 -> 2
- net I2C1_SDA: track 0.00 -> 36.5 mm, vias 0 -> 4
- net SPI2_MOSI: track 1.62 -> 38.1 mm, vias 0 -> 2
- net AI_CRNT: track 0.00 -> 33.6 mm, vias 0 -> 4
- net GPIO_PB8: track 0.00 -> 31.8 mm, vias 0 -> 2
- net I2C1_SCL: track 0.00 -> 31.5 mm, vias 0 -> 4
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- added copper zone on F.Cu, net +3V3
- added copper zone on In2.Cu, net +3V3
- added copper zone on In1.Cu, net GND
- removed copper zone on In1.Cu, net +3V3
- removed copper zone on In2.Cu, net +5V
Other:
- board text added: "3V3"
- board text added: "5V"
- board text added: "PB8"
- board text added: "RST"
